Commit message: camera added feed working but IK not working

File: src/akabot_description/urdf/end_effector_camera.xacro (robot description, xacro)
@@ -27,6 +27,5 @@
     <parent link="claw_base"/>
     <child link="ee_camera_link"/>
-    <!-- Position: slightly forward and down from claw_base -->
-    <origin xyz="0.015 0.04 -0.01" rpy="0 ${pi/2} 0"/>
+    <origin xyz="0.025 0.035 -0.03" rpy="0 ${pi/2} 0"/>
   </joint>
   <!-- Optical frame for the camera -->
@@ -37,21 +36,24 @@
     <origin xyz="0 0 0" rpy="${-pi/2} 0 ${-pi/2}"/>
   </joint>
-  <!-- Gazebo plugin for end effector camera -->
-  <xacro:property name="deg_to_rad" value="0.01745329252" />
+  <!-- ==========================================
+       GAZEBO SIM (IGNITION) CAMERA SENSOR
+       This uses the NEW Gazebo plugin system
+       ========================================== -->
   <gazebo reference="ee_camera_link">
     <sensor name="ee_camera" type="camera">
-      <pose>0 0 0 0 0 0</pose>
+      <always_on>1</always_on>
+      <update_rate>30</update_rate>
       <visualize>true</visualize>
-      <update_rate>30</update_rate>
+      <topic>ee_camera</topic>
       <camera>
-        <horizontal_fov>${60*deg_to_rad}</horizontal_fov>
+        <horizontal_fov>1.2217</horizontal_fov> <!-- 70 degrees -->
         <image>
-          <format>R8G8B8</format>
           <width>640</width>
           <height>480</height>
+          <format>R8G8B8</format>
         </image>
         <clip>
-          <near>0.01</near>
-          <far>2.0</far>
+          <near>0.02</near>
+          <far>3.0</far>
         </clip>
         <noise>
@@ -61,13 +63,4 @@
         </noise>
       </camera>
-      <plugin name="ee_camera_controller" filename="libgazebo_ros_camera.so">
-        <ros>
-          <namespace>/ee_camera</namespace>
-          <remapping>image_raw:=image_raw</remapping>
-          <remapping>camera_info:=camera_info</remapping>
-        </ros>
-        <frame_name>ee_camera_optical_link</frame_name>
-        <hack_baseline>0.07</hack_baseline>
-      </plugin>
     </sensor>
   </gazebo>
