Commit message: Fix arm to sit on table: correct top_plate_joint z offset from 0.15 to 0.048

File: src/akabot_description/urdf/akabot_core.xacro (robot description, xacro)
@@ -40,5 +40,5 @@
     <parent link="base_plate"/>
     <child link="top_plate"/>
-    <origin rpy="0 0 1.5" xyz="0.0 0 0.15"/>
+    <origin rpy="0 0 1.5" xyz="0.0 0 0.048"/>
     <axis xyz="0 0 1" />
     <limit effort="1000.0" lower="1.56" upper="4.68" velocity="1.0" />

Commit message: Fix arm description: align base_plate at origin (0,0,0) to sit properly on table

File: src/akabot_description/urdf/akabot_core.xacro (robot description, xacro)
@@ -14,5 +14,5 @@
     <parent link="base_link"/>
     <child link="base_plate"/>
-    <origin xyz="0.1 0.05 0"/>
+    <origin xyz="0 0 0"/>
   </joint>
   <!-- Base plate -->
@@ -40,5 +40,5 @@
     <parent link="base_plate"/>
     <child link="top_plate"/>
-    <origin rpy="0 0 1.5" xyz="0.0 0 0.048"/>
+    <origin rpy="0 0 1.5" xyz="0 0 0.048"/>
     <axis xyz="0 0 1" />
     <limit effort="1000.0" lower="1.56" upper="4.68" velocity="1.0" />
