Commit message: trajectory is generated using MoveIt and arm is reaches the target pose successfully.

File: install/akabot_description/share/akabot_description/urdf/akabot_core.xacro (robot description, xacro)
@@ -40,5 +40,5 @@
     <parent link="base_plate"/>
     <child link="top_plate"/>
-    <origin rpy="0 0 1.5" xyz="0.0 0 0.048"/>
+    <origin rpy="0 0 1.5" xyz="0.0 0 0.15"/>
     <axis xyz="0 0 1" />
     <limit effort="1000.0" lower="1.56" upper="4.68" velocity="1.0" />
